File: kicad_hiltop_lora_board/lora_board.kicad_pcb (KiCad board)
At the start: 4 copper layers, 159.9 x 99.9 mm, 36 parts, among them J3 Conn_03x32_DIN41612, U13 CP2102N-A01-GQFN24

Commit message: finished design - Rev A
Parts:
- removed C52: DNF, Capacitor_SMD:C_0603_1608Metric
- removed C55: 4.7uF, Capacitor_SMD:C_0402_1005Metric
- removed C56: 100nF, Capacitor_SMD:C_0402_1005Metric
- removed R76, R79, R80, R83, R84: 0R, Resistor_SMD:R_0603_1608Metric
- removed R77: DNF, Resistor_SMD:R_0603_1608Metric
- removed R78: 24K, Resistor_SMD:R_0603_1608Metric
- removed R81, R82: 330R, Resistor_SMD:R_0603_1608Metric
- removed the REF** at (82.1, 133.2)
- removed TP31, TP32, TP33, TP34, TP35, TP36: Test_Point, TestPoint:TestPoint_THTPad_D1.0mm_Drill0.5mm
- removed U13: CP2102N-A01-GQFN24, Package_DFN_QFN:QFN-24-1EP_4x4mm_P0.5mm_EP2.6x2.6mm_ThermalVias
- added C1: 100nF, Capacitor_SMD:C_0603_1608Metric, F.Cu at (161.0, 64.5)
- added C2: 10uF, Capacitor_SMD:C_0805_2012Metric, F.Cu at (79.3, 132.3)
- added C3: 10uF, Capacitor_SMD:C_0805_2012Metric, F.Cu at (92.8, 129.4)
- added C4: 100nF, Capacitor_SMD:C_0603_1608Metric, F.Cu at (81.0, 105.5)
- added C5: 100uF, Capacitor_SMD:CP_Elec_6.3x7.7, F.Cu at (98.8, 131.2)
- added C6: DNF, Capacitor_SMD:C_0603_1608Metric, F.Cu at (86.2, 67.3)
- added C7: 4.7uF, Capacitor_SMD:C_0603_1608Metric, F.Cu at (83.2, 63.0)
- added C8: 100nF, Capacitor_SMD:C_0603_1608Metric, F.Cu at (81.2, 63.0)
- added C9: 100nF, Capacitor_SMD:C_0603_1608Metric, F.Cu at (171.8, 98.0)
- added D1: MBR230LSFT1G, Diode_SMD:D_SOD-123, F.Cu at (86.1, 133.0)
- added JP1: Jumper_NC_Dual, Connector_PinHeader_2.54mm:PinHeader_1x03_P2.54mm_Vertical, F.Cu at (78.0, 124.0)
- added R1: 0R, Resistor_SMD:R_0603_1608Metric, F.Cu at (172.2, 63.0)
- added R10: DNF, Resistor_SMD:R_0603_1608Metric, F.Cu at (88.0, 115.7)
- added R11: 0R, Resistor_SMD:R_0603_1608Metric, F.Cu at (83.5, 67.2)
- added R12: DNF, Resistor_SMD:R_0603_1608Metric, F.Cu at (88.0, 67.3)
- added R13: 24K, Resistor_SMD:R_0603_1608Metric, F.Cu at (78.8, 65.8)
- added R14: 47K, Resistor_SMD:R_0603_1608Metric, F.Cu at (83.5, 65.5)
- added R15: 0R, Resistor_SMD:R_0603_1608Metric, F.Cu at (96.0, 68.2)
- added R16: DNF, Resistor_SMD:R_0603_1608Metric, F.Cu at (96.0, 66.2)
- added R17: DNF, Resistor_SMD:R_0603_1608Metric, F.Cu at (96.0, 64.2)
- added R18: DNF, Resistor_SMD:R_0603_1608Metric, F.Cu at (96.0, 62.2)
- added R19: DNF, Resistor_SMD:R_0603_1608Metric, F.Cu at (169.8, 98.0)
- added R2: 0R, Resistor_SMD:R_0603_1608Metric, F.Cu at (169.8, 63.0)
- added R21: DNF, Resistor_SMD:R_0603_1608Metric, F.Cu at (154.8, 129.8)
- added R22: DNF, Resistor_SMD:R_0603_1608Metric, F.Cu at (163.0, 129.2)
- added R23: DNF, Resistor_SMD:R_0603_1608Metric, F.Cu at (162.7, 98.2)
- added R24: DNF, Resistor_SMD:R_0603_1608Metric, F.Cu at (154.7, 96.7)
- added R25: DNF, Resistor_SMD:R_0603_1608Metric, F.Cu at (159.5, 129.0)
- added R3: 0R, Resistor_SMD:R_0603_1608Metric, F.Cu at (167.2, 63.0)
- added R4: 0R, Resistor_SMD:R_0603_1608Metric, F.Cu at (164.8, 63.0)
- added R5: DNF, Resistor_SMD:R_0603_1608Metric, F.Cu at (170.8, 87.2)
- added R6: 0R, Resistor_SMD:R_0603_1608Metric, F.Cu at (168.8, 84.5)
- added R7: 10K, Resistor_SMD:R_0603_1608Metric, F.Cu at (83.0, 114.0)
- added R8: 4K7, Resistor_SMD:R_0603_1608Metric, F.Cu at (84.0, 102.0)
- added R9: 4K7, Resistor_SMD:R_0603_1608Metric, F.Cu at (85.5, 116.4)
- added REF**: OSHW-Logo2_9.8x8mm_SilkScreen, Symbol:OSHW-Logo2_9.8x8mm_SilkScreen, F.Cu at (117.1, 134.3)
- added TP1: Test_Point, TestPoint:TestPoint_THTPad_D1.0mm_Drill0.5mm, F.Cu at (79.0, 68.8)
- added TP10: Test_Point, TestPoint:TestPoint_THTPad_D1.0mm_Drill0.5mm, F.Cu at (104.2, 62.2)
- added TP3: Test_Point, TestPoint:TestPoint_THTPad_D1.0mm_Drill0.5mm, F.Cu at (109.5, 55.5)
- added TP4: Test_Point, TestPoint:TestPoint_THTPad_D1.0mm_Drill0.5mm, F.Cu at (107.0, 53.5)
- added TP5: Test_Point, TestPoint:TestPoint_THTPad_D1.0mm_Drill0.5mm, F.Cu at (112.5, 58.2)
- added TP6: Test_Point, TestPoint:TestPoint_THTPad_D1.0mm_Drill0.5mm, F.Cu at (115.0, 60.5)
- added TP7: Test_Point, TestPoint:TestPoint_THTPad_D1.0mm_Drill0.5mm, F.Cu at (104.2, 68.5)
- added TP8: Test_Point, TestPoint:TestPoint_THTPad_D1.0mm_Drill0.5mm, F.Cu at (104.2, 66.5)
- added TP9: Test_Point, TestPoint:TestPoint_THTPad_D1.0mm_Drill0.5mm, F.Cu at (104.2, 64.2)
- added U1: ERIC-LORA, Devtank_PCB_Lib:eRIC-LoRa_RF_Module, F.Cu at (167.2, 74.8)
- added U2: LD1117S33TR_SOT223, Package_TO_SOT_SMD:SOT-223-3_TabPin2, F.Cu at (86.0, 127.8)
- added U3: AT25DN512CSSHF-B, Package_SO:SOIC-8_3.9x4.9mm_P1.27mm, F.Cu at (86.0, 108.5)
- added U4: CP2102N-A01-GQFN24, Package_DFN_QFN:QFN-24-1EP_4x4mm_P0.5mm_EP2.6x2.6mm_ThermalVias, F.Cu at (87.2, 60.8)
- added U5: XBee_SMT, RF_Module:Digi_XBee_SMT, F.Cu at (163.8, 113.8)
- R20: value 47K -> DNF
- moved R20 67.0 mm to (167.5, 98.0), turned to 270 degrees
- moved TP2 66.7 mm to (176.2, 63.5), turned to 0 degrees
- moved REF** 35.0 mm to (129.8, 134.5)
- moved G*** 26.9 mm to (203.8, 121.2)
- moved REF** 21.9 mm to (201.2, 68.8)
- moved TP14 1.69 mm to (69.7, 119.3)
- renumbered J3 to J1, TP101 to TP11, TP102 to TP12, TP103 to TP13, TP104 to TP14, TP105 to TP15
Connections:
- J1 pad 30b: (no net) -> /USB_DATA_N
- J1 pad 31b: (no net) -> /USB_DATA_P
- R20 pad 1: GND -> /HOST_TX
- TP2 pad 1: /RESET -> Net-(TP2-Pad1)
Routing:
- net +3V3: track 8.53 -> 320.3 mm, vias 2 -> 7
- net /HOST_CTS: track 0.00 -> 203.5 mm, vias 0 -> 2
- net /HOST_RTS: track 0.00 -> 194.9 mm, vias 0 -> 2
- net /HOST_TX: track 0.00 -> 150.1 mm, vias 0 -> 2
- net /HOST_RX: track 0.00 -> 147.5 mm, vias 0 -> 1
- net /RESET: track 11.7 -> 116.0 mm
- net +5V: track 8.03 -> 107.7 mm, vias 1 -> 0
- net /HOST_SLEEP: track 0.00 -> 88.9 mm, vias 0 -> 1
- net /PORT_SEL: track 0.00 -> 56.7 mm, vias 0 -> 1
- net +3V3_LOC: track 0.00 -> 30.1 mm
- net /SPI0_MOSI: track 0.00 -> 29.8 mm
- net /SPI0_CLK: track 0.00 -> 26.0 mm
- net /SPI0_MISO: track 0.00 -> 25.3 mm, vias 0 -> 1
- net (no net): track 20.4 -> 0.00 mm, vias 2 -> 0
- net GND: track 7.06 -> 25.6 mm, vias 33 -> 51
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- removed copper zone on In2.Cu, net +3V3
- removed copper zone on In1.Cu, net GND
- removed copper zone on In2.Cu, net GND
Other:
- board size 159.9 x 99.9 mm -> 159.4 x 99.9 mm
- copper layers 4 -> 2
- board text added: "IoT Board"
- board text added: "PN: 304-011"
- board text removed: "Moto Board"
- board text removed: "PN: 304-008"
