File: kicad_hiltop_lora_board/lora_board.sch (KiCad schematic (older format))
At the start: 25 parts, among them J3 Conn_03x32_DIN41612, U2 LD1117S33TR_SOT223, U3 AT25DN512CSSHF-B

Commit message: finished design - Rev A
Parts:
- added C1, C9: 100nF, Capacitor_SMD:C_0603_1608Metric, symbol lora_board-rescue:C-device-Sensi_Board-rescue-Motor_Control_Board-rescue-moto_b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
- added R1, R2, R3, R4, R6: 0R, Resistor_SMD:R_0603_1608Metric, symbol lora_board-rescue:R-device-Sensi_Board-rescue-Motor_Control_Board-rescue-moto_b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
- added R19, R20, R21, R22, R23, R24, R25, R5: DNF, Resistor_SMD:R_0603_1608Metric, symbol lora_board-rescue:R-device-Sensi_Board-rescue-Motor_Control_Board-rescue-moto_b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
- added TP2, TP5, TP6: Test_Point, TestPoint:TestPoint_THTPad_D1.0mm_Drill0.5mm, symbol lora_board-rescue:Test_Point-Connector-Sensi_Board-rescue-Motor_Control_Board-r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
- added U1: ERIC-LORA, Devtank_PCB_Lib:eRIC-LoRa_RF_Module, symbol Devtank:ERIC-LORA
- added U5: XBee_SMT, RF_Module:Digi_XBee_SMT, symbol rfcom:XBee_SMT
- C4: renamed from C12; footprint Capacitor_SMD:C_0402_1005Metric -> Capacitor_SMD:C_0603_1608Metric
- renumbered C10 to C2, C11 to C3, C13 to C5, D32 to D1, J3 to J1, R17 to R10, R14 to R7, R15 to R8, R16 to R9, TP2 to TP1, TP36 to TP10, TP101 to TP11, TP102 to TP12, TP103 to TP13, TP104 to TP14, TP105 to TP15, TP31 to TP3, TP32 to TP4, TP33 to TP7, TP34 to TP8, TP35 to TP9
Connections:
- net +3V3: now also C1.2, C9.2, R25.1, U1.6 (VCC), U5.2 (VCC)
- net GND: now also C1.1, C9.1, R5.2, U1.23 (RF_GND), U1.7 (GND), U5.1 (GND), U5.11 (GND), U5.13 (GND), U5.22 (GND), U5.35 (GND)
- net RESET: now also R23.1
- net STM_BOOT0 renamed HOST_SLEEP
- net HOST_SLEEP: now also R24.1, R6.2
- net STM_DEBUG_RX renamed HOST_RX
- net HOST_RX: now also R19.1, R2.1
- net STM_DEBUG_TX renamed HOST_TX
- net HOST_TX: now also R20.1, R3.1
- net STM_RES1 renamed USB_Debug/GPIO1
- net STM_RES2 renamed USB_Debug/GPIO0
- net STM_RESET renamed USB_Debug/GPIO2
- new net: TP2.1, U1.1 (GPIO)
- new net: R24.2, U5.10 (DIO8/SLEEP_REQUEST)
- new net: R21.2, U5.25 (DIO7/~CTS)
- new net: R25.2, U5.27 (VREF)
- new net: R22.2, U5.29 (DIO6/~RTS)
- new net: R19.2, U5.3 (DIO13/UART_TX)
- new net: R20.2, U5.4 (DIO14/UART_RX/~CONFIG)
- new net: R23.2, U5.6 (RESET/OD_OUT)
- new net HOST_CTS: R1.1, R21.1, TP6.1
- new net HOST_RTS: R22.1, R4.1, TP5.1
- new net LORA_CTS: R1.2, U1.2 (BUSY)
- new net LORA_RTS: R4.2, U1.5 (HOST_RDY)
- new net LORA_RX: R2.2, U1.3 (SDO)
- new net LORA_SLEEP: R5.1, R6.1, U1.17 (SLEEP)
- new net LORA_TX: R3.2, U1.4 (SDI)
- no-connect marks 59 -> 76
Other:
- note added: "Lora Wireless Module (Option 1)\nLPRS eRIC-LoRa"
- note added: "XBee Wireless Module (Option 2)\nDigi XB24CZ7UIS-004"
- moved on the sheet: C2, C3, C4, C5, D1, J1A, J1B, J1C, JP1, R10, R7, R8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
